File: hardware/pcb/furuta_pendulum.kicad_pcb (KiCad board)
At the start: 4 copper layers, 34 x 55 mm, 70 parts, among them J2 LCD_ST7735S, J3 DRV8313, J5 Conn_ARM_SWD_TagConnect_TC2030, J7 Encoders, J8 USB_C_Receptacle_USB2.0_14P, U1 AMS1117-3.3, U3 USBLC6-2SC6, U7 ATSAMD51J20A-A

Commit message: update
Parts:
- removed C25: 100n, Capacitor_SMD:C_0402_1005Metric
- removed TP10, TP11, TP7, TP8, TP9: TestPoint, TestPoint:TestPoint_Pad_D1.5mm
- added C27: 100n, Capacitor_SMD:C_0402_1005Metric, F.Cu at (131.7, 67.1)
- added C28: 100n, Capacitor_SMD:C_0402_1005Metric, F.Cu at (131.7, 60.0)
- added TP6: TestPoint, TestPoint:TestPoint_Pad_D1.5mm, F.Cu at (159.9, 34.0)
- D1, D2, J8, U7: moved to B.Cu
- moved TP4 71.5 mm to (159.9, 26.9)
- moved TP5 54.8 mm to (159.9, 30.5)
- moved FID3 45.7 mm to (127.9, 33.0)
- moved TP1 41.4 mm to (159.9, 23.4)
- moved FID1 40.2 mm to (131.3, 32.4)
- moved R22 36.7 mm to (160.8, 77.1)
- moved R24 36.7 mm to (160.8, 72.1)
- moved R25 36.7 mm to (160.8, 69.6)
- moved R23 36.7 mm to (160.8, 74.6)
- moved J2 31.5 mm to (121.9, 50.1)
- moved J7 30.3 mm to (149.8, 52.6)
- moved J5 29.4 mm to (129.7, 49.2)
- moved FID2 28.9 mm to (124.1, 33.6)
- moved R16 21.6 mm to (113.5, 59.2)
- moved R17 21.6 mm to (111.0, 59.0)
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Connections:
- net /unconnected-(J8-SHIELD-PadSH)_2_2 renamed /unconnected-(J8-SHIELD-PadSH)_2
Routing:
- net /MCU_RESET: track 46.1 -> 0.00 mm, vias 2 -> 0
- net /DRV_FAULT: track 38.6 -> 0.00 mm, vias 1 -> 0
- net +3.3V: track 37.3 -> 0.00 mm, vias 15 -> 0
- net VBUS: track 35.7 -> 0.00 mm, vias 3 -> 0
- net GND: track 35.1 -> 0.00 mm, vias 126 -> 0
- net /MCU_SW2: track 33.4 -> 0.00 mm, vias 2 -> 0
- net Net-(J5-SWO): track 32.8 -> 0.00 mm, vias 2 -> 0
- net +12VF: track 31.4 -> 0.00 mm, vias 7 -> 0
- net /DRV_ENABLE: track 29.2 -> 0.00 mm, vias 1 -> 0
- net /DRV_PWM3: track 29.0 -> 0.00 mm, vias 1 -> 0
- net /DRV_SLEEP: track 28.9 -> 0.00 mm, vias 1 -> 0
- net /DRV_PWM1: track 28.9 -> 0.00 mm, vias 1 -> 0
- net /DRV_RESET: track 28.8 -> 0.00 mm, vias 1 -> 0
- net /DRV_PWM2: track 28.1 -> 0.00 mm, vias 1 -> 0
- net /VDDIO: track 26.8 -> 0.00 mm
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- removed copper zone on In2.Cu, net +12VF
- removed copper zone on In2.Cu, net +3.3V
- removed copper zone on B.Cu, net GND
- removed copper zone on F.Cu, net GND
- removed copper zone on In1.Cu, net GND
- removed copper zone on B.Cu, net PGND
- removed copper zone on F.Cu, net PGND
- removed copper zone on In1.Cu, net PGND
Other:
- board size 34 x 55 mm -> 32 x 55 mm
- board text removed: "Furuta Pendulum Control Board"
- board text removed: "Rev 1, 06/26 By: Morten Vandborg"
