File: hardware/pcb/furuta_pendulum.kicad_sch (KiCad schematic)
At the start: 70 parts, among them J2 LCD_ST7735S, J3 DRV8313, J5 Conn_ARM_SWD_TagConnect_TC2030, J7 Encoders, J8 USB_C_Receptacle_USB2.0_14P, U1 AMS1117-3.3, U3 USBLC6-2SC6, U7 ATSAMD51J20A-A

Commit message: update
Parts:
- removed TP10, TP11, TP7, TP8, TP9: TestPoint, TestPoint:TestPoint_Pad_D1.5mm, symbol Connector:TestPoint
- added C27, C28: 100n, Capacitor_SMD:C_0402_1005Metric, symbol Device:C
- added C29: 10u, Capacitor_SMD:C_0805_2012Metric, symbol Device:C
- added TP6: TestPoint, TestPoint:TestPoint_Pad_D1.5mm, symbol Connector:TestPoint
- C25: now not fitted; now left out of the parts list
Connections:
- net +3.3V: now also C29.2
- net GND: now also C27.1, C28.1, C29.1
- net PGND: now also TP6.1
- net VDDIO: now also C27.2, C28.2
Other:
- note removed: "There are already 10uF at AMS1117-3.3"
- moved on the sheet: C19, C22, C26, FB3
